File: PCB/SofleKeyboard.sch (KiCad schematic (older format))
At the start: 85 parts, among them J1 LED, J2 4PIN, J3 OLED, P1 i2c_pin, P2 i2c_pin, SW1 SW_PUSH, SW10 SW_PUSH, SW11 SW_PUSH, SW12 SW_PUSH, SW13 SW_PUSH, SW14 SW_PUSH, SW15 SW_PUSH, SW16 SW_PUSH, SW17 SW_PUSH, SW18 SW_PUSH, SW19 SW_PUSH, SW2 SW_PUSH, SW20 SW_PUSH, SW21 SW_PUSH, SW22 SW_PUSH, SW23 SW_PUSH, SW24 SW_PUSH, SW25 Rotary_Encoder_Switch, SW26 SW_PUSH, SW27 SW_PUSH, SW28 SW_PUSH, SW29 SW_PUSH, SW3 SW_PUSH, SW30 SW_PUSH, SW4 SW_PUSH, SW5 SW_PUSH, SW6 SW_PUSH, SW7 SW_PUSH, SW8 SW_PUSH, SW9 SW_PUSH, U1 ProMicro

Commit message: Added CRKBDv3 style SK6812-E LEDs and panelization
Parts:
- removed JP1, JP2, JP3, JP4, JP5, JP6, JP7, JP8: Jumper_NO_Small, SofleKeyboard-footprint:Jumper, symbol Device:Jumper_NO_Small
- removed W1: jumper, SofleKeyboard-footprint:jumper_data, symbol Device:Jumper
- added D31, D32, D33, D34, D35, D36, D37, D38, D39, D40, D41, D42, D43, D44, D45, D46, D47, D48, D49, D50, D51, D52, D53, D54, D55, D56, D57, D58, D59, D60: D, SofleKeyboard-footprint:Diode_SOD123, symbol SofleKeyboard-rescue:D-Lily58-cache-Lily58_Pro-rescue
- added J4: OLED, SofleKeyboard-footprint:OLED_4Pin, symbol SofleKeyboard-rescue:OLED-Lily58-cache-Lily58_Pro-rescue
- added J5: 4PIN, SofleKeyboard-footprint:MJ-4PP-9, symbol SofleKeyboard-rescue:MJ-4PP-9-Lily58-cache-Lily58_Pro-rescue
- added J6: LED, SofleKeyboard-footprint:LED, symbol SofleKeyboard-rescue:LED-Lily58-cache-Lily58_Pro-rescue
- added LED1, LED10, LED11, LED12, LED13, LED14, LED15, LED16, LED17, LED18, LED19, LED2, LED20, LED21, LED22, LED23, LED24, LED25, LED26, LED27, LED28, LED29, LED3, LED30, LED31, LED32, LED33, LED34, LED35, LED36, LED37, LED38, LED39, LED4, LED40, LED41, LED42, LED43, LED44, LED45, LED46, LED47, LED48, LED49, LED5, LED50, LED51, LED52, LED53, LED54, LED55, LED56, LED57, LED58, LED59, LED6, LED60, LED61, LED62, LED63, LED64, LED65, LED66, LED67, LED68, LED69, LED7, LED70, LED71, LED72, LED73, LED74, LED8, LED9: YS-SK6812MINI-E, CRKBD:YS-SK6812MINI-E, symbol CRKBD:YS-SK6812MINI-E
- added P3, P4: i2c_pin, SofleKeyboard-footprint:1pin_conn, symbol SofleKeyboard-rescue:i2c_pin-Lily58-cache-Lily58_Pro-rescue
- added R3, R4: R, SofleKeyboard-footprint:RESISTOR_mini, symbol SofleKeyboard-rescue:R-Lily58-cache-Lily58_Pro-rescue
- added RSW2: SW_RST, SofleKeyboard-footprint:TACT_SWITCH_TVBP06, symbol SofleKeyboard-rescue:SW_RST-Lily58-cache-Lily58_Pro-rescue
- added SW31: Rotary_Encoder_Switch, SofleKeyboard-footprint:RotaryEncoder_Alps_EC11E-Switch_Vertical_H20mm-keebio_modified, symbol Device:Rotary_Encoder_Switch
- added SW32, SW33, SW34, SW35, SW36, SW37, SW38, SW39, SW41, SW42, SW43, SW44, SW45, SW46, SW47, SW48, SW49, SW50, SW51, SW52, SW53, SW54, SW55, SW56, SW57, SW58, SW59, SW60: SW_PUSH, SofleKeyboard-footprint:CherryMX_KailhLowProfile_Hotswap, symbol SofleKeyboard-rescue:SW_PUSH-Lily58-cache-Lily58_Pro-rescue
- added SW40: SW_PUSH, SofleKeyboard-footprint:CherryMX_KailhLowProfile_Hotswap_1.5, symbol SofleKeyboard-rescue:SW_PUSH-Lily58-cache-Lily58_Pro-rescue
- added TH10, TH11, TH12, TH13, TH14, TH9: HOLE, SofleKeyboard-footprint:HOLE_M2_TH, symbol SofleKeyboard-rescue:HOLE-Lily58-cache-Lily58_Pro-rescue
- added TH8: HOLE, SofleKeyboard-footprint:M2_HOLE_PCB, symbol SofleKeyboard-rescue:HOLE-Lily58-cache-Lily58_Pro-rescue
- added U2: ProMicro, SofleKeyboard-footprint:ProMicro, symbol SofleKeyboard-rescue:ProMicro_2-Lily58-cache-Lily58_Pro-rescue
- renumbered D26 to D10, D3 to D11, D9 to D12, D15 to D13, D21 to D14, D27 to D15, D4 to D16, D10 to D17, D16 to D18, D22 to D19, D7 to D2, D28 to D20, D5 to D21, D11 to D22, D17 to D23, D23 to D24, D29 to D25, D6 to D26, D12 to D27, D18 to D28, D24 to D29, D13 to D3, D19 to D4, D25 to D5, D2 to D6, D8 to D7, D14 to D8, D20 to D9, J3 to J1, J1 to J3, SW25 to SW1, SW26 to SW10, SW3 to SW11, SW9 to SW12, SW15 to SW13, SW21 to SW14, SW27 to SW15, SW4 to SW16, SW10 to SW17, SW16 to SW18, SW22 to SW19, SW1 to SW2, SW28 to SW20, SW5 to SW21, SW11 to SW22, SW17 to SW23, SW23 to SW24, SW29 to SW25, SW6 to SW26, SW12 to SW27, SW18 to SW28, SW24 to SW29, SW7 to SW3, SW13 to SW4, SW19 to SW5, SW2 to SW6, SW8 to SW7, SW14 to SW8, SW20 to SW9
Connections:
- net labels added: DATA_L, ENCA_L, ENCB_L, GNDA, LED_L, RESET_L, SCL_L, SDA_L, SW25A_L, SW25B_L, VDD, col0_L, col1_L, col2_L, col3_L, col4_L, col5_L, i2c_c_L, i2c_d_L, row0_L, row1_L, row2_L, row3_L, row4_L
- wire segments 87 -> 460
- no-connect marks 2 -> 4
Other:
- moved on the sheet: D1, D10, D11, D12, D13, D14, D15, D16, D17, D18, D19, D2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
