File: PCB/SofleKeyboard.kicad_pcb (KiCad board)
At the start: 2 copper layers, 137.2 x 109.2 mm, 87 parts, among them J1 LED, J2 4PIN, J3 OLED, P1 i2c_pin, P2 i2c_pin, SW1 SW_PUSH, SW10 SW_PUSH, SW11 SW_PUSH, SW12 SW_PUSH, SW13 SW_PUSH, SW14 SW_PUSH, SW15 SW_PUSH, SW16 SW_PUSH, SW17 SW_PUSH, SW18 SW_PUSH, SW19 SW_PUSH, SW2 SW_PUSH, SW20 SW_PUSH, SW21 SW_PUSH, SW22 SW_PUSH, SW23 SW_PUSH, SW24 SW_PUSH, SW25 Rotary_Encoder_Switch, SW26 SW_PUSH, SW27 SW_PUSH, SW28 SW_PUSH, SW29 SW_PUSH, SW3 SW_PUSH, SW30 SW_PUSH, SW4 SW_PUSH, SW5 SW_PUSH, SW6 SW_PUSH, SW7 SW_PUSH, SW8 SW_PUSH, SW9 SW_PUSH, U1 ProMicro

Commit message: Added CRKBDv3 style SK6812-E LEDs and panelization
Parts:
- removed JP1, JP2, JP3, JP4, JP5, JP6, JP7, JP8: Jumper_NO_Small, SofleKeyboard-footprint:Jumper
- removed Ref** (x2): Val**, SofleKeyboard-footprint:SofleLogoSmall
- added D31: D, SofleKeyboard-footprint:Diode_SOD123, B.Cu at (151.9, 84.0)
- added D32: D, SofleKeyboard-footprint:Diode_SOD123, B.Cu at (151.9, 105.2)
- added D33: D, SofleKeyboard-footprint:Diode_SOD123, B.Cu at (151.9, 121.9)
- added D34: D, SofleKeyboard-footprint:Diode_SOD123, B.Cu at (151.9, 143.3)
- added D35: D, SofleKeyboard-footprint:Diode_SOD123, B.Cu at (170.2, 128.3)
- added D36: D, SofleKeyboard-footprint:Diode_SOD123, B.Cu at (132.6, 82.8)
- added D37: D, SofleKeyboard-footprint:Diode_SOD123, B.Cu at (132.6, 102.6)
- added D38: D, SofleKeyboard-footprint:Diode_SOD123, B.Cu at (132.6, 121.9)
- added D39: D, SofleKeyboard-footprint:Diode_SOD123, B.Cu at (132.6, 141.2)
- added D40: D, SofleKeyboard-footprint:Diode_SOD123, B.Cu at (172.1, 149.8)
- added D41: D, SofleKeyboard-footprint:Diode_SOD123, B.Cu at (113.8, 84.3)
- added D42: D, SofleKeyboard-footprint:Diode_SOD123, B.Cu at (113.8, 103.1)
- added D43: D, SofleKeyboard-footprint:Diode_SOD123, B.Cu at (113.8, 121.2)
- added D44: D, SofleKeyboard-footprint:Diode_SOD123, B.Cu at (113.8, 141.2)
- added D45: D, SofleKeyboard-footprint:Diode_SOD123, B.Cu at (151.4, 165.1)
- added D46: D, SofleKeyboard-footprint:Diode_SOD123, B.Cu at (94.5, 84.8)
- added D47: D, SofleKeyboard-footprint:Diode_SOD123, B.Cu at (94.5, 104.1)
- added D48: D, SofleKeyboard-footprint:Diode_SOD123, B.Cu at (95.0, 121.9)
- added D49: D, SofleKeyboard-footprint:Diode_SOD123, B.Cu at (94.5, 143.3)
- added D50: D, SofleKeyboard-footprint:Diode_SOD123, B.Cu at (124.0, 160.5)
- added D51: D, SofleKeyboard-footprint:Diode_SOD123, B.Cu at (75.2, 86.0)
- added D52: D, SofleKeyboard-footprint:Diode_SOD123, B.Cu at (75.2, 108.2)
- added D53: D, SofleKeyboard-footprint:Diode_SOD123, B.Cu at (75.7, 124.6)
- added D54: D, SofleKeyboard-footprint:Diode_SOD123, B.Cu at (75.7, 146.3)
- added D55: D, SofleKeyboard-footprint:Diode_SOD123, B.Cu at (105.2, 160.5)
- added D56: D, SofleKeyboard-footprint:Diode_SOD123, B.Cu at (58.4, 90.6)
- added D57: D, SofleKeyboard-footprint:Diode_SOD123, B.Cu at (58.4, 109.4)
- added D58: D, SofleKeyboard-footprint:Diode_SOD123, B.Cu at (58.4, 128.5)
- added D59: D, SofleKeyboard-footprint:Diode_SOD123, B.Cu at (58.4, 147.8)
- added D60: D, SofleKeyboard-footprint:Diode_SOD123, B.Cu at (85.9, 164.6)
- added J4: OLED, SofleKeyboard-footprint:OLED_4Pin, F.Cu at (185.2, 105.1)
- added J5: 4PIN, SofleKeyboard-footprint:MJ-4PP-9, F.Cu at (194.3, 118.1)
- added J6: LED, SofleKeyboard-footprint:LED, B.Cu at (172.7, 106.7)
- added LED1: YS-SK6812MINI-E, CRKBD:YS-SK6812MINI-E, B.Cu at (238.8, 161.0)
- added LED10: YS-SK6812MINI-E, CRKBD:YS-SK6812MINI-E, B.Cu at (286.5, 122.4)
- added LED11: YS-SK6812MINI-E, CRKBD:YS-SK6812MINI-E, B.Cu at (305.8, 127.0)
- added LED12: YS-SK6812MINI-E, CRKBD:YS-SK6812MINI-E, B.Cu at (325.1, 128.5)
- added LED13: YS-SK6812MINI-E, CRKBD:YS-SK6812MINI-E, B.Cu at (325.1, 148.8)
- added LED14: YS-SK6812MINI-E, CRKBD:YS-SK6812MINI-E, B.Cu at (305.8, 146.3)
- added LED15: YS-SK6812MINI-E, CRKBD:YS-SK6812MINI-E, B.Cu at (267.7, 120.9)
- added LED16: YS-SK6812MINI-E, CRKBD:YS-SK6812MINI-E, B.Cu at (248.4, 122.4)
- added LED17: YS-SK6812MINI-E, CRKBD:YS-SK6812MINI-E, B.Cu at (230.1, 124.5)
- added LED18: YS-SK6812MINI-E, CRKBD:YS-SK6812MINI-E, B.Cu at (229.6, 105.7)
- added LED19: YS-SK6812MINI-E, CRKBD:YS-SK6812MINI-E, B.Cu at (248.9, 103.1)
- added LED2: YS-SK6812MINI-E, CRKBD:YS-SK6812MINI-E, B.Cu at (258.6, 160.5)
- added LED20: YS-SK6812MINI-E, CRKBD:YS-SK6812MINI-E, B.Cu at (325.1, 89.9)
- added LED21: YS-SK6812MINI-E, CRKBD:YS-SK6812MINI-E, B.Cu at (325.1, 109.2)
- added LED22: YS-SK6812MINI-E, CRKBD:YS-SK6812MINI-E, B.Cu at (305.8, 108.2)
- added LED23: YS-SK6812MINI-E, CRKBD:YS-SK6812MINI-E, B.Cu at (286.5, 103.1)
- added LED24: YS-SK6812MINI-E, CRKBD:YS-SK6812MINI-E, B.Cu at (267.7, 102.1)
- added LED25: YS-SK6812MINI-E, CRKBD:YS-SK6812MINI-E, B.Cu at (305.8, 87.9)
- added LED26: YS-SK6812MINI-E, CRKBD:YS-SK6812MINI-E, B.Cu at (287.0, 83.8)
- added LED27: YS-SK6812MINI-E, CRKBD:YS-SK6812MINI-E, B.Cu at (267.2, 82.3)
- added LED28: YS-SK6812MINI-E, CRKBD:YS-SK6812MINI-E, B.Cu at (248.9, 83.3)
- added LED29: YS-SK6812MINI-E, CRKBD:YS-SK6812MINI-E, B.Cu at (229.6, 85.9)
- added LED3: YS-SK6812MINI-E, CRKBD:YS-SK6812MINI-E, B.Cu at (277.4, 161.5)
- added LED30: YS-SK6812MINI-E, CRKBD:YS-SK6812MINI-E, F.Cu at (296.7, 148.8)
- added LED31: YS-SK6812MINI-E, CRKBD:YS-SK6812MINI-E, F.Cu at (267.7, 144.3)
- added LED32: YS-SK6812MINI-E, CRKBD:YS-SK6812MINI-E, F.Cu at (226.6, 148.3)
- added LED33: YS-SK6812MINI-E, CRKBD:YS-SK6812MINI-E, F.Cu at (230.1, 128.5)
- added LED34: YS-SK6812MINI-E, CRKBD:YS-SK6812MINI-E, F.Cu at (325.1, 113.3)
- added LED35: YS-SK6812MINI-E, CRKBD:YS-SK6812MINI-E, F.Cu at (305.8, 92.5)
- added LED36: YS-SK6812MINI-E, CRKBD:YS-SK6812MINI-E, F.Cu at (267.2, 86.4)
- added LED37: YS-SK6812MINI-E, CRKBD:YS-SK6812MINI-E, F.Cu at (229.6, 89.9)
- added LED38: YS-SK6812MINI-E, CRKBD:YS-SK6812MINI-E, B.Cu at (94.5, 165.6)
- added LED39: YS-SK6812MINI-E, CRKBD:YS-SK6812MINI-E, B.Cu at (113.8, 161.5)
- added LED4: YS-SK6812MINI-E, CRKBD:YS-SK6812MINI-E, B.Cu at (296.7, 165.6)
- added LED40: YS-SK6812MINI-E, CRKBD:YS-SK6812MINI-E, B.Cu at (132.6, 160.5)
- added LED41: YS-SK6812MINI-E, CRKBD:YS-SK6812MINI-E, B.Cu at (152.4, 162.6)
- added LED42: YS-SK6812MINI-E, CRKBD:YS-SK6812MINI-E, B.Cu at (181.4, 165.1)
- added LED43: YS-SK6812MINI-E, CRKBD:YS-SK6812MINI-E, B.Cu at (161.5, 143.8)
- added LED44: YS-SK6812MINI-E, CRKBD:YS-SK6812MINI-E, B.Cu at (142.2, 141.7)
- added LED45: YS-SK6812MINI-E, CRKBD:YS-SK6812MINI-E, B.Cu at (123.4, 140.7)
- added LED46: YS-SK6812MINI-E, CRKBD:YS-SK6812MINI-E, B.Cu at (104.1, 142.2)
- added LED47: YS-SK6812MINI-E, CRKBD:YS-SK6812MINI-E, B.Cu at (85.3, 146.3)
- added LED48: YS-SK6812MINI-E, CRKBD:YS-SK6812MINI-E, B.Cu at (66.0, 148.8)
- added LED49: YS-SK6812MINI-E, CRKBD:YS-SK6812MINI-E, B.Cu at (66.0, 128.5)
- added LED5: YS-SK6812MINI-E, CRKBD:YS-SK6812MINI-E, B.Cu at (209.8, 165.1)
- added LED50: YS-SK6812MINI-E, CRKBD:YS-SK6812MINI-E, B.Cu at (85.3, 127.0)
- added LED51: YS-SK6812MINI-E, CRKBD:YS-SK6812MINI-E, B.Cu at (104.6, 122.4)
- added LED52: YS-SK6812MINI-E, CRKBD:YS-SK6812MINI-E, B.Cu at (123.4, 120.9)
- added LED53: YS-SK6812MINI-E, CRKBD:YS-SK6812MINI-E, B.Cu at (142.7, 122.4)
- added LED54: YS-SK6812MINI-E, CRKBD:YS-SK6812MINI-E, B.Cu at (161.0, 124.5)
- added LED55: YS-SK6812MINI-E, CRKBD:YS-SK6812MINI-E, B.Cu at (161.5, 105.7)
- added LED56: YS-SK6812MINI-E, CRKBD:YS-SK6812MINI-E, B.Cu at (142.2, 103.1)
- added LED57: YS-SK6812MINI-E, CRKBD:YS-SK6812MINI-E, B.Cu at (123.4, 102.1)
- added LED58: YS-SK6812MINI-E, CRKBD:YS-SK6812MINI-E, B.Cu at (104.6, 103.1)
- added LED59: YS-SK6812MINI-E, CRKBD:YS-SK6812MINI-E, B.Cu at (85.3, 108.2)
- added LED6: YS-SK6812MINI-E, CRKBD:YS-SK6812MINI-E, B.Cu at (229.6, 143.8)
- added LED60: YS-SK6812MINI-E, CRKBD:YS-SK6812MINI-E, B.Cu at (66.0, 109.2)
- added LED61: YS-SK6812MINI-E, CRKBD:YS-SK6812MINI-E, B.Cu at (66.0, 89.9)
- added LED62: YS-SK6812MINI-E, CRKBD:YS-SK6812MINI-E, B.Cu at (85.3, 87.9)
- added LED63: YS-SK6812MINI-E, CRKBD:YS-SK6812MINI-E, B.Cu at (104.1, 83.8)
- added LED64: YS-SK6812MINI-E, CRKBD:YS-SK6812MINI-E, B.Cu at (124.0, 82.3)
- added LED65: YS-SK6812MINI-E, CRKBD:YS-SK6812MINI-E, B.Cu at (142.2, 83.3)
- added LED66: YS-SK6812MINI-E, CRKBD:YS-SK6812MINI-E, B.Cu at (161.5, 85.9)
- added LED67: YS-SK6812MINI-E, CRKBD:YS-SK6812MINI-E, F.Cu at (94.5, 148.8)
- added LED68: YS-SK6812MINI-E, CRKBD:YS-SK6812MINI-E, F.Cu at (123.4, 144.3)
- added LED69: YS-SK6812MINI-E, CRKBD:YS-SK6812MINI-E, F.Cu at (164.6, 148.3)
- added LED7: YS-SK6812MINI-E, CRKBD:YS-SK6812MINI-E, B.Cu at (248.9, 141.7)
- added LED70: YS-SK6812MINI-E, CRKBD:YS-SK6812MINI-E, F.Cu at (161.0, 128.5)
- added LED71: YS-SK6812MINI-E, CRKBD:YS-SK6812MINI-E, F.Cu at (66.0, 113.3)
- added LED72: YS-SK6812MINI-E, CRKBD:YS-SK6812MINI-E, F.Cu at (85.3, 92.5)
- added LED73: YS-SK6812MINI-E, CRKBD:YS-SK6812MINI-E, F.Cu at (124.0, 86.4)
- added LED74: YS-SK6812MINI-E, CRKBD:YS-SK6812MINI-E, F.Cu at (161.5, 89.9)
- added LED8: YS-SK6812MINI-E, CRKBD:YS-SK6812MINI-E, B.Cu at (267.7, 140.7)
- added LED9: YS-SK6812MINI-E, CRKBD:YS-SK6812MINI-E, B.Cu at (287.0, 142.2)
- added P3: i2c_pin, SofleKeyboard-footprint:1pin_conn, F.Cu at (179.2, 110.8)
- added P4: i2c_pin, SofleKeyboard-footprint:1pin_conn, F.Cu at (179.2, 108.6)
- added R3: R, SofleKeyboard-footprint:RESISTOR_mini, F.Cu at (183.9, 110.8)
- added R4: R, SofleKeyboard-footprint:RESISTOR_mini, F.Cu at (183.9, 108.5)
- added RSW2: SW_RST, SofleKeyboard-footprint:TACT_SWITCH_TVBP06, F.Cu at (191.9, 108.0)
- added SW31: Rotary_Encoder_Switch, SofleKeyboard-footprint:RotaryEncoder_Alps_EC11E-Switch_Vertical_H20mm-keebio_modified, F.Cu at (181.9, 135.0)
- added SW32: SW_PUSH, SofleKeyboard-footprint:CherryMX_KailhLowProfile_Hotswap, F.Cu at (161.4, 80.5)
- added SW33: SW_PUSH, SofleKeyboard-footprint:CherryMX_KailhLowProfile_Hotswap, F.Cu at (161.4, 99.6)
- added SW34: SW_PUSH, SofleKeyboard-footprint:CherryMX_KailhLowProfile_Hotswap, F.Cu at (161.4, 118.6)
- added SW35: SW_PUSH, SofleKeyboard-footprint:CherryMX_KailhLowProfile_Hotswap, F.Cu at (161.4, 137.6)
- added SW36: SW_PUSH, SofleKeyboard-footprint:CherryMX_KailhLowProfile_Hotswap, F.Cu at (142.4, 78.1)
- added SW37: SW_PUSH, SofleKeyboard-footprint:CherryMX_KailhLowProfile_Hotswap, F.Cu at (142.4, 97.2)
- added SW38: SW_PUSH, SofleKeyboard-footprint:CherryMX_KailhLowProfile_Hotswap, F.Cu at (142.4, 116.2)
- added SW39: SW_PUSH, SofleKeyboard-footprint:CherryMX_KailhLowProfile_Hotswap, F.Cu at (142.4, 135.3)
- added SW40: SW_PUSH, SofleKeyboard-footprint:CherryMX_KailhLowProfile_Hotswap_1.5, F.Cu at (176.0, 160.6)
- added SW41: SW_PUSH, SofleKeyboard-footprint:CherryMX_KailhLowProfile_Hotswap, F.Cu at (123.3, 76.7)
- added SW42: SW_PUSH, SofleKeyboard-footprint:CherryMX_KailhLowProfile_Hotswap, F.Cu at (123.3, 95.8)
- added SW43: SW_PUSH, SofleKeyboard-footprint:CherryMX_KailhLowProfile_Hotswap, F.Cu at (123.3, 114.9)
- added SW44: SW_PUSH, SofleKeyboard-footprint:CherryMX_KailhLowProfile_Hotswap, F.Cu at (123.3, 133.9)
- added SW45: SW_PUSH, SofleKeyboard-footprint:CherryMX_KailhLowProfile_Hotswap, F.Cu at (154.1, 156.9)
- added SW46: SW_PUSH, SofleKeyboard-footprint:CherryMX_KailhLowProfile_Hotswap, F.Cu at (104.3, 78.1)
- added SW47: SW_PUSH, SofleKeyboard-footprint:CherryMX_KailhLowProfile_Hotswap, F.Cu at (104.3, 97.1)
- added SW48: SW_PUSH, SofleKeyboard-footprint:CherryMX_KailhLowProfile_Hotswap, F.Cu at (104.3, 116.2)
- added SW49: SW_PUSH, SofleKeyboard-footprint:CherryMX_KailhLowProfile_Hotswap, F.Cu at (104.3, 135.3)
- added SW50: SW_PUSH, SofleKeyboard-footprint:CherryMX_KailhLowProfile_Hotswap, F.Cu at (132.9, 154.2)
- added SW51: SW_PUSH, SofleKeyboard-footprint:CherryMX_KailhLowProfile_Hotswap, F.Cu at (85.2, 82.9)
- added SW52: SW_PUSH, SofleKeyboard-footprint:CherryMX_KailhLowProfile_Hotswap, F.Cu at (85.2, 101.8)
- added SW53: SW_PUSH, SofleKeyboard-footprint:CherryMX_KailhLowProfile_Hotswap, F.Cu at (85.2, 121.0)
- added SW54: SW_PUSH, SofleKeyboard-footprint:CherryMX_KailhLowProfile_Hotswap, F.Cu at (85.2, 140.0)
- added SW55: SW_PUSH, SofleKeyboard-footprint:CherryMX_KailhLowProfile_Hotswap, F.Cu at (113.8, 154.2)
- added SW56: SW_PUSH, SofleKeyboard-footprint:CherryMX_KailhLowProfile_Hotswap, F.Cu at (66.2, 84.4)
- added SW57: SW_PUSH, SofleKeyboard-footprint:CherryMX_KailhLowProfile_Hotswap, F.Cu at (66.2, 103.3)
- added SW58: SW_PUSH, SofleKeyboard-footprint:CherryMX_KailhLowProfile_Hotswap, F.Cu at (66.2, 122.5)
- added SW59: SW_PUSH, SofleKeyboard-footprint:CherryMX_KailhLowProfile_Hotswap, F.Cu at (66.2, 141.5)
- added SW60: SW_PUSH, SofleKeyboard-footprint:CherryMX_KailhLowProfile_Hotswap, F.Cu at (94.7, 158.4)
- added TH10: HOLE, SofleKeyboard-footprint:HOLE_M2_TH, B.Cu at (152.3, 90.1)
- added TH11: HOLE, SofleKeyboard-footprint:HOLE_M2_TH, B.Cu at (76.1, 92.3)
- added TH12: HOLE, SofleKeyboard-footprint:HOLE_M2_TH, B.Cu at (152.3, 128.1)
- added TH13: HOLE, SofleKeyboard-footprint:HOLE_M2_TH, B.Cu at (76.1, 130.5)
- added TH14: HOLE, SofleKeyboard-footprint:HOLE_M2_TH, B.Cu at (176.9, 145.3)
- added TH8: HOLE, SofleKeyboard-footprint:M2_HOLE_PCB, B.Cu at (190.4, 124.0)
- added TH9: HOLE, SofleKeyboard-footprint:M2_HOLE_PCB, B.Cu at (174.9, 124.0)
- added U2: ProMicro, SofleKeyboard-footprint:ProMicro, F.Cu at (181.6, 86.4)
- W1: moved to B.Cu
- moved D19 133.5 mm to (296.7, 143.3), turned to 90 degrees
- moved D22 133.2 mm to (316.0, 108.2), turned to 90 degrees
- moved D17 133.2 mm to (296.7, 104.1), turned to 90 degrees
- moved D14 133.0 mm to (277.4, 141.2), turned to 90 degrees
- moved D12 132.9 mm to (277.4, 103.1), turned to 90 degrees
- moved D24 132.7 mm to (315.5, 146.3), turned to 90 degrees
- moved D4 132.4 mm to (239.3, 143.3), turned to 90 degrees
- moved D2 132.4 mm to (239.3, 105.2), turned to 90 degrees
- moved D30 132.4 mm to (305.3, 164.6), turned to 90 degrees
- moved D20 132.1 mm to (267.2, 160.5), turned to 90 degrees
- moved D25 131.8 mm to (286.0, 160.5), turned to 90 degrees
- moved D9 131.0 mm to (258.6, 141.2), turned to 90 degrees
- moved D7 130.9 mm to (258.6, 102.6), turned to 90 degrees
- moved D16 128.5 mm to (296.7, 84.8), turned to 90 degrees
- moved D11 128.5 mm to (277.4, 84.3), turned to 90 degrees
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- renumbered D26 to D10, D3 to D11, D9 to D12, D15 to D13, D21 to D14, D27 to D15, D4 to D16, D10 to D17, D16 to D18, D22 to D19, D7 to D2, D28 to D20, D5 to D21, D11 to D22, D17 to D23, D23 to D24, D29 to D25, D6 to D26, D12 to D27, D18 to D28, D24 to D29, D13 to D3, D19 to D4, D25 to D5, D2 to D6, D8 to D7, D14 to D8, D20 to D9, J3 to J1, J1 to J3, SW25 to SW1, SW26 to SW10, SW3 to SW11, SW9 to SW12, SW15 to SW13, SW21 to SW14, SW27 to SW15, SW4 to SW16, SW10 to SW17, SW16 to SW18, SW22 to SW19, SW1 to SW2, SW28 to SW20, SW5 to SW21, SW11 to SW22, SW17 to SW23, SW23 to SW24, SW29 to SW25, SW6 to SW26, SW12 to SW27, SW18 to SW28, SW24 to SW29, SW7 to SW3, SW13 to SW4, SW19 to SW5, SW2 to SW6, SW8 to SW7, SW14 to SW8, SW20 to SW9
Connections:
- J1 pad 1: Net-(J3-Pad1) -> SDA
- J1 pad 2: Net-(J3-Pad2) -> SCL
- J1 pad 3: Net-(J3-Pad3) -> VCC
- J1 pad 4: Net-(J3-Pad4) -> GND
- J2 pad 3: /i2c_d -> DATA
- P2 pad 1: /i2c_d -> DATA
Routing:
- net col0: track 358.0 -> 0.00 mm, vias 11 -> 0
- net col1: track 350.6 -> 0.00 mm, vias 11 -> 0
- net col2: track 334.4 -> 0.00 mm, vias 11 -> 0
- net col3: track 314.7 -> 0.00 mm, vias 11 -> 0
- net col4: track 311.0 -> 0.00 mm, vias 11 -> 0
- net SW25A: track 206.1 -> 0.00 mm, vias 9 -> 0
- net row3: track 170.1 -> 0.00 mm, vias 1 -> 0
- net row2: track 165.8 -> 0.00 mm, vias 1 -> 0
- net row4: track 152.5 -> 0.00 mm, vias 1 -> 0
- net row1: track 138.3 -> 0.00 mm, vias 1 -> 0
- net row0: track 138.2 -> 0.00 mm, vias 1 -> 0
- net GND: track 124.4 -> 0.00 mm, vias 45 -> 0
- net VCC: track 74.2 -> 0.00 mm, vias 3 -> 0
- net ENCB: track 73.1 -> 0.00 mm, vias 1 -> 0
- net ENCA: track 69.0 -> 0.00 mm, vias 1 -> 0
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- added copper zone on B.Cu, net (none)
- added copper zone on F.Cu, net (none)
Other:
- board size 137.2 x 109.2 mm -> 278.2 x 109.2 mm
- board text removed: "Sofle Keyboard v1 by Josef Adamcik"

Commit message: Cleaned up stray edges in pcb
Parts:
- SW10, SW40: footprint SofleKeyboard-footprint:CherryMX_KailhLowProfile_Hotswap_1.5 -> CRKBD:CherryMX_Hotswap_1.5u
- SW11, SW12, SW13, SW14, SW15, SW16, SW17, SW18, SW19, SW2, SW20, SW21, SW22, SW23, SW24, SW25, SW26, SW27, SW28, SW29, SW3, SW30, SW32, SW33, SW34, SW35, SW36, SW37, SW38, SW39, SW4, SW41, SW42, SW43, SW44, SW45, SW46, SW47, SW48, SW49, SW5, SW50, SW51, SW52, SW53, SW54, SW55, SW56, SW57, SW58, SW59, SW6, SW60, SW7, SW8, SW9: footprint SofleKeyboard-footprint:CherryMX_KailhLowProfile_Hotswap -> CRKBD:CherryMX_Hotswap

Commit message: Panelized PCB
Parts:
- added REF**: Breakaway_Tabs, CRKBD:Breakaway_Tabs, F.Cu at (261.0, 163.5)
- added REF**: Breakaway_Tabs, CRKBD:Breakaway_Tabs, F.Cu at (131.0, 163.5)
- added REF**: Breakaway_Tabs, CRKBD:Breakaway_Tabs, F.Cu at (111.0, 67.8)
- added REF**: Breakaway_Tabs, CRKBD:Breakaway_Tabs, F.Cu at (153.5, 67.7)
- added REF**: Breakaway_Tabs, CRKBD:Breakaway_Tabs, F.Cu at (235.0, 67.8)
- added REF**: Breakaway_Tabs, CRKBD:Breakaway_Tabs, F.Cu at (284.6, 67.8)
- moved LED42 2.55 mm to (181.6, 162.6)
- moved LED5 2.55 mm to (209.6, 162.6)
- moved D20 1.30 mm to (268.0, 159.5)
- moved D50 1.12 mm to (123.5, 159.5)
- moved LED40 1.11 mm to (133.0, 159.5)
- moved LED2 0.78 mm to (258.0, 160.0)
Other:
- board size 278.2 x 109.2 mm -> 278.2 x 123 mm
